File: psi3214_spice_dispositivo.kicad_sch (KiCad schematic)
At the start: 16 parts, among them U2 ${SIM.PARAMS}, U3 ${SIM.PARAMS}

Commit message: minor updates
Parts:
- C2: value 100n -> 1u
- R11: value 27k -> 22k
- R5: value 47k -> 1k
- R6: value 100k -> 220
- R9: value 6.8k -> 1k
Connections:
- net entrada: now reaches C2.1, R3.1
- net saida_amp1: now reaches C3.1, R6.1, R7.1, U2.5
- net saida_filtro: now reaches C3.2, R7.2, R8.2, U3.1 (+)
- net saida_cap: now reaches C2.2, R4.2, U2.1 (+)
- net out_general renamed saida
Other:
- note added: "$$A_v = 1 + \frac{R11}{R9}$$"
- note added: "$$A_v = 1 + \frac{R6}{R5}$$"
- note added: "AmpOp não inversor"
- note added: "fc = 16Hz Remove DC"
- moved on the sheet: R4
